File: EE-Ink-Power.sch (KiCad schematic (older format))
At the start: 64 parts, among them J1 USB_A, Q4 IRLML6402, Q5 IRLML6402, Q6 IRLML6402, U5 LM358, U6 MCP73831, U7 MCP1825S, U8 LT1945, U9 LT1945

Commit message: Began linking footprints to the components.
Parts:
- C10, C11, C12, C13, C14, C15, C16, C17, C18, C19, C6, C7, C8, C9: footprint (none) -> Capacitors_SMD:C_0805
- D4: footprint (none) -> LEDs:LED_0805
- D5: footprint (none) -> SMD_Packages-Custom:DO-214AA
- J1: footprint (none) -> Connectors-Custom3:SMT-Micro-USB-AB
- Q4, Q5, Q6: footprint (none) -> TO_SOT_Packages_SMD:SOT-23
- R15, R16, R17, R18, R19, R20, R21, R22, R23, R24, R25, R26, R27, R28, R29, R30, R31: footprint (none) -> Resistors_SMD:R_0805
- U5: footprint (none) -> Housings_SOIC:SOIC-8_3.9x4.9mm_Pitch1.27mm
- U7: footprint (none) -> TO_SOT_Packages_SMD:SOT-223
- U8, U9: footprint (none) -> Housings_SSOP:MSOP-10_3x3mm_Pitch0.5mm
Changed lines of the file:
@@
 F 0 "U8" H 7350 2900 60  0000 C CNN
 F 1 "LT1945" H 7800 2350 60  0000 C CNN
-F 2 "" H 7800 2350 60  0001 C CNN
+F 2 "Housings_SSOP:MSOP-10_3x3mm_Pitch0.5mm" H 7800 2350 60  0001 C CNN
 F 3 "" H 7800 2350 60  0001 C CNN
 	1    7800 2350
@@
 F 0 "Q5" V 6150 1700 50  0000 L CNN
 F 1 "IRLML6402" V 6450 1400 50  0000 L CNN
-F 2 "" H 6400 1700 50  0001 C CNN
+F 2 "TO_SOT_Packages_SMD:SOT-23" H 6400 1700 50  0001 C CNN
 F 3 "" H 6200 1600 50  0001 C CNN
 	1    6200 1600
@@
 F 0 "C12" H 6700 1800 50  0000 L CNN
 F 1 "4u7" H 6850 1650 50  0000 L CNN
-F 2 "" H 6800 1700 50  0001 C CNN
+F 2 "Capacitors_SMD:C_0805" H 6800 1700 50  0001 C CNN
 F 3 "" H 6800 1700 50  0001 C CNN
 	1    6800 1700
@@
 F 0 "R20" V 5800 1750 50  0000 C CNN
 F 1 "12k" V 5900 1750 50  0000 C CNN
-F 2 "" V 5830 1750 50  0001 C CNN
+F 2 "Resistors_SMD:R_0805" V 5830 1750 50  0001 C CNN
 F 3 "" H 5900 1750 50  0001 C CNN
 	1    5900 1750
@@
 F 0 "R21" V 5800 2400 50  0000 C CNN
 F 1 "47k" V 5900 2400 50  0000 C CNN
-F 2 "" V 5830 2400 50  0001 C CNN
+F 2 "Resistors_SMD:R_0805" V 5830 2400 50  0001 C CNN
 F 3 "" H 5900 2400 50  0001 C CNN
 	1    5900 2400
@@
 F 0 "C14" V 8550 1300 50  0000 L CNN
 F 1 "100nF" V 8650 1550 50  0000 L CNN
-F 2 "" H 8600 1500 50  0001 C CNN
+F 2 "Capacitors_SMD:C_0805" H 8600 1500 50  0001 C CNN
 F 3 "" H 8600 1500 50  0001 C CNN
 	1    8600 1500
@@
 F 0 "R28" V 9600 1800 50  0000 C CNN
 F 1 "402k" V 9700 1800 50  0000 C CNN
-F 2 "" V 9630 1800 50  0001 C CNN
+F 2 "Resistors_SMD:R_0805" V 9630 1800 50  0001 C CNN
 F 3 "" H 9700 1800 50  0001 C CNN
 	1    9700 1800
@@
 F 0 "C18" H 9300 1950 50  0000 L CNN
 F 1 "100pF" H 9400 1750 50  0000 L CNN
-F 2 "" H 9400 1850 50  0001 C CNN
+F 2 "Capacitors_SMD:C_0805" H 9400 1850 50  0001 C CNN
 F 3 "" H 9400 1850 50  0001 C CNN
 	1    9400 1850
@@
 F 0 "R29" V 9600 2450 50  0000 C CNN
 F 1 "38k3" V 9700 2450 50  0000 C CNN
-F 2 "" V 9630 2450 50  0001 C CNN
+F 2 "Resistors_SMD:R_0805" V 9630 2450 50  0001 C CNN
 F 3 "" H 9700 2450 50  0001 C CNN
 	1    9700 2450
@@
 F 0 "C16" H 8900 2900 50  0000 L CNN
 F 1 "4p7" H 9000 2700 50  0000 L CNN
-F 2 "" H 9000 2800 50  0001 C CNN
+F 2 "Capacitors_SMD:C_0805" H 9000 2800 50  0001 C CNN
 F 3 "" H 9000 2800 50  0001 C CNN
 	1    9000 2800
@@
 F 0 "R24" V 9300 2800 50  0000 C CNN
 F 1 "402k" V 9400 2800 50  0000 C CNN
-F 2 "" V 9330 2800 50  0001 C CNN
+F 2 "Resistors_SMD:R_0805" V 9330 2800 50  0001 C CNN
 F 3 "" H 9400 2800 50  0001 C CNN
 	1    9400 2800
@@
 F 0 "R25" V 9300 3250 50  0000 C CNN
 F 1 "36k" V 9400 3250 50  0000 C CNN
-F 2 "" V 9330 3250 50  0001 C CNN
+F 2 "Resistors_SMD:R_0805" V 9330 3250 50  0001 C CNN
 F 3 "" H 9400 3250 50  0001 C CNN
 	1    9400 3250
@@
 F 0 "D5" H 8350 3200 50  0000 C CNN
 F 1 "SS24" H 8350 3000 50  0000 C CNN
-F 2 "" H 8350 3100 50  0001 C CNN
+F 2 "SMD_Packages-Custom:DO-214AA" H 8350 3100 50  0001 C CNN
 F 3 "" H 8350 3100 50  0001 C CNN
 	1    8350 3100
@@
 F 0 "U9" H 7350 5500 60  0000 C CNN
 F 1 "LT1945" H 7800 4950 60  0000 C CNN
-F 2 "" H 7800 4950 60  0001 C CNN
+F 2 "Housings_SSOP:MSOP-10_3x3mm_Pitch0.5mm" H 7800 4950 60  0001 C CNN
 F 3 "" H 7800 4950 60  0001 C CNN
 	1    7800 4950
@@
 F 0 "Q6" V 6150 4300 50  0000 L CNN
 F 1 "IRLML6402" V 6450 4000 50  0000 L CNN
-F 2 "" H 6400 4300 50  0001 C CNN
+F 2 "TO_SOT_Packages_SMD:SOT-23" H 6400 4300 50  0001 C CNN
 F 3 "" H 6200 4200 50  0001 C CNN
 	1    6200 4200
@@
 F 0 "C13" H 6700 4400 50  0000 L CNN
 F 1 "4u7" H 6850 4250 50  0000 L CNN
-F 2 "" H 6800 4300 50  0001 C CNN
+F 2 "Capacitors_SMD:C_0805" H 6800 4300 50  0001 C CNN
 F 3 "" H 6800 4300 50  0001 C CNN
 	1    6800 4300
@@
 F 0 "R22" V 5800 4350 50  0000 C CNN
 F 1 "12k" V 5900 4350 50  0000 C CNN
-F 2 "" V 5830 4350 50  0001 C CNN
+F 2 "Resistors_SMD:R_0805" V 5830 4350 50  0001 C CNN
 F 3 "" H 5900 4350 50  0001 C CNN
 	1    5900 4350
@@
 F 0 "R23" V 5800 5000 50  0000 C CNN
 F 1 "47k" V 5900 5000 50  0000 C CNN
-F 2 "" V 5830 5000 50  0001 C CNN
+F 2 "Resistors_SMD:R_0805" V 5830 5000 50  0001 C CNN
 F 3 "" H 5900 5000 50  0001 C CNN
 	1    5900 5000
@@
 F 0 "C15" V 8550 3900 50  0000 L CNN
 F 1 "100nF" V 8650 4150 50  0000 L CNN
-F 2 "" H 8600 4100 50  0001 C CNN
+F 2 "Capacitors_SMD:C_0805" H 8600 4100 50  0001 C CNN
 F 3 "" H 8600 4100 50  0001 C CNN
 	1    8600 4100
@@
 F 0 "R30" V 9600 4400 50  0000 C CNN
 F 1 "470k" V 9700 4400 50  0000 C CNN
-F 2 "" V 9630 4400 50  0001 C CNN
+F 2 "Resistors_SMD:R_0805" V 9630 4400 50  0001 C CNN
 F 3 "" H 9700 4400 50  0001 C CNN
 	1    9700 4400
@@
 F 0 "C19" H 9300 4550 50  0000 L CNN
 F 1 "100pF" H 9400 4350 50  0000 L CNN
-F 2 "" H 9400 4450 50  0001 C CNN
+F 2 "Capacitors_SMD:C_0805" H 9400 4450 50  0001 C CNN
 F 3 "" H 9400 4450 50  0001 C CNN
 	1    9400 4450
@@
 F 0 "R31" V 9600 5050 50  0000 C CNN
 F 1 "33k" V 9700 5050 50  0000 C CNN
-F 2 "" V 9630 5050 50  0001 C CNN
+F 2 "Resistors_SMD:R_0805" V 9630 5050 50  0001 C CNN
 F 3 "" H 9700 5050 50  0001 C CNN
 	1    9700 5050
@@
 F 0 "C17" H 8900 5500 50  0000 L CNN
 F 1 "4p7" H 9000 5300 50  0000 L CNN
-F 2 "" H 9000 5400 50  0001 C CNN
+F 2 "Capacitors_SMD:C_0805" H 9000 5400 50  0001 C CNN
 F 3 "" H 9000 5400 50  0001 C CNN
 	1    9000 5400
@@
 F 0 "R26" V 9300 5400 50  0000 C CNN
 F 1 "560k" V 9400 5400 50  0000 C CNN
-F 2 "" V 9330 5400 50  0001 C CNN
+F 2 "Resistors_SMD:R_0805" V 9330 5400 50  0001 C CNN
 F 3 "" H 9400 5400 50  0001 C CNN
 	1    9400 5400
@@
 F 0 "R27" V 9300 5850 50  0000 C CNN
 F 1 "33k" V 9400 5850 50  0000 C CNN
-F 2 "" V 9330 5850 50  0001 C CNN
+F 2 "Resistors_SMD:R_0805" V 9330 5850 50  0001 C CNN
 F 3 "" H 9400 5850 50  0001 C CNN
 	1    9400 5850
@@
 F 0 "Q4" V 5050 5450 50  0000 L CNN
 F 1 "IRLML6402" V 5350 5150 50  0000 L CNN
-F 2 "" H 5300 5450 50  0001 C CNN
+F 2 "TO_SOT_Packages_SMD:SOT-23" H 5300 5450 50  0001 C CNN
 F 3 "" H 5100 5350 50  0001 C CNN
 	1    5100 5350
@@
 F 0 "C9" H 3660 5670 50  0000 L CNN
 F 1 "4u7" H 3650 5500 50  0000 L CNN
-F 2 "" H 3650 5600 50  0001 C CNN
+F 2 "Capacitors_SMD:C_0805" H 3650 5600 50  0001 C CNN
 F 3 "" H 3650 5600 50  0001 C CNN
 	1    3650 5600
@@
 F 0 "C11" H 4760 5620 50  0000 L CNN
 F 1 "1uF" H 4750 5450 50  0000 L CNN
-F 2 "" H 4750 5550 50  0001 C CNN
+F 2 "Capacitors_SMD:C_0805" H 4750 5550 50  0001 C CNN
 F 3 "" H 4750 5550 50  0001 C CNN
 	1    4750 5550
@@
 F 0 "U5" H 2000 5400 50  0000 L CNN
 F 1 "LM358" H 2000 5000 50  0000 L CNN
-F 2 "" H 2000 5200 50  0001 C CNN
+F 2 "Housings_SOIC:SOIC-8_3.9x4.9mm_Pitch1.27mm" H 2000 5200 50  0001 C CNN
 F 3 "" H 2000 5200 50  0001 C CNN
 	1    2000 5200
@@
 F 0 "R15" V 1150 5500 50  0000 C CNN
 F 1 "200k" V 1250 5500 50  0000 C CNN
-F 2 "" V 1180 5500 50  0001 C CNN
+F 2 "Resistors_SMD:R_0805" V 1180 5500 50  0001 C CNN
 F 3 "" H 1250 5500 50  0001 C CNN
 	1    1250 5500
@@
 F 0 "C8" H 2710 5470 50  0000 L CNN
 F 1 "100nF" H 2710 5320 50  0000 L CNN
-F 2 "" H 2700 5400 50  0001 C CNN
+F 2 "Capacitors_SMD:C_0805" H 2700 5400 50  0001 C CNN
 F 3 "" H 2700 5400 50  0001 C CNN
 	1    2700 5400
@@
 F 0 "J1" H 1850 3200 50  0000 L CNN
 F 1 "USB_A" H 1850 3100 50  0000 L CNN
-F 2 "" H 2200 2700 50  0001 C CNN
+F 2 "Connectors-Custom3:SMT-Micro-USB-AB" H 2200 2700 50  0001 C CNN
 F 3 "" H 2200 2700 50  0001 C CNN
 	1    2050 2750
@@
 F 0 "R18" V 3000 2750 50  0000 C CNN
 F 1 "470" V 3100 2750 50  0000 C CNN
-F 2 "" V 3030 2750 50  0001 C CNN
+F 2 "Resistors_SMD:R_0805" V 3030 2750 50  0001 C CNN
 F 3 "" H 3100 2750 50  0001 C CNN
 	1    3100 2750
@@
 F 0 "D4" V 3000 3050 50  0000 L CNN
 F 1 "LED_Small" H 2925 2950 50  0001 L CNN
-F 2 "" V 3100 3050 50  0001 C CNN
+F 2 "LEDs:LED_0805" V 3100 3050 50  0001 C CNN
 F 3 "" V 3100 3050 50  0001 C CNN
 	1    3100 3050
@@
 F 0 "R19" V 4100 2950 50  0000 C CNN
 F 1 "2k" V 4200 2950 50  0000 C CNN
-F 2 "" V 4130 2950 50  0001 C CNN
+F 2 "Resistors_SMD:R_0805" V 4130 2950 50  0001 C CNN
 F 3 "" H 4200 2950 50  0001 C CNN
 	1    4200 2950
@@
 F 0 "C10" H 4410 2770 50  0000 L CNN
 F 1 "4u7" H 4400 2600 50  0000 L CNN
-F 2 "" H 4400 2700 50  0001 C CNN
+F 2 "Capacitors_SMD:C_0805" H 4400 2700 50  0001 C CNN
 F 3 "" H 4400 2700 50  0001 C CNN
 	1    4400 2700
@@
 F 0 "R16" V 2500 3100 50  0000 C CNN
 F 1 "27" V 2400 3100 50  0000 C CNN
-F 2 "" V 2330 3100 50  0001 C CNN
+F 2 "Resistors_SMD:R_0805" V 2330 3100 50  0001 C CNN
 F 3 "" H 2400 3100 50  0001 C CNN
 	1    2400 3100
@@
 F 0 "R17" V 2400 3100 50  0000 C CNN
 F 1 "27" V 2500 3100 50  0000 C CNN
-F 2 "" V 2430 3100 50  0001 C CNN
+F 2 "Resistors_SMD:R_0805" V 2430 3100 50  0001 C CNN
 F 3 "" H 2500 3100 50  0001 C CNN
 	1    2500 3100
@@
 F 0 "C6" H 1300 2850 50  0000 L CNN
 F 1 "100nF" H 1400 2700 50  0000 L CNN
-F 2 "" H 1400 2750 50  0001 C CNN
+F 2 "Capacitors_SMD:C_0805" H 1400 2750 50  0001 C CNN
 F 3 "" H 1400 2750 50  0001 C CNN
 	1    1400 2750
@@
 F 0 "C7" H 1600 2850 50  0000 L CNN
 F 1 "4u7" H 1700 2700 50  0000 L CNN
-F 2 "" H 1700 2750 50  0001 C CNN
+F 2 "Capacitors_SMD:C_0805" H 1700 2750 50  0001 C CNN
 F 3 "" H 1700 2750 50  0001 C CNN
 	1    1700 2750
@@
 F 0 "U7" H 4400 5000 60  0000 C CNN
 F 1 "MCP1825S" H 4200 5350 60  0000 C CNN
-F 2 "" H 4100 5200 60  0001 C CNN
+F 2 "TO_SOT_Packages_SMD:SOT-223" H 4100 5200 60  0001 C CNN
 F 3 "" H 4100 5200 60  0001 C CNN
 	1    4200 5250

Commit message: Created footprint for the connector of the E-ink display and linked it.
Parts:
- D10, D6, D7, D8, D9: footprint (none) -> SMD_Packages-Custom:DO-214AA
- L1, L2, L3, L4: footprint (none) -> Resistors_SMD:R_0805
Changed lines of the file:
@@
 F 0 "L3" V 7750 1500 50  0000 C CNN
 F 1 "22uH" V 7875 1500 50  0000 C CNN
-F 2 "" H 7800 1500 50  0001 C CNN
+F 2 "Resistors_SMD:R_0805" H 7800 1500 50  0001 C CNN
 F 3 "" H 7800 1500 50  0001 C CNN
 	1    7800 1500
@@
 F 0 "D7" H 8900 1900 50  0000 C CNN
 F 1 "SS24" H 8900 1700 50  0000 C CNN
-F 2 "" H 8900 1800 50  0001 C CNN
+F 2 "SMD_Packages-Custom:DO-214AA" H 8900 1800 50  0001 C CNN
 F 3 "" H 8900 1800 50  0001 C CNN
 	1    8900 1800
@@
 F 0 "L1" V 7200 3100 50  0000 C CNN
 F 1 "22uH" V 7325 3100 50  0000 C CNN
-F 2 "" H 7250 3100 50  0001 C CNN
+F 2 "Resistors_SMD:R_0805" H 7250 3100 50  0001 C CNN
 F 3 "" H 7250 3100 50  0001 C CNN
 	1    7250 3100
@@
 F 0 "D9" H 9150 1600 50  0000 C CNN
 F 1 "SS24" H 9150 1400 50  0000 C CNN
-F 2 "" H 9150 1500 50  0001 C CNN
+F 2 "SMD_Packages-Custom:DO-214AA" H 9150 1500 50  0001 C CNN
 F 3 "" H 9150 1500 50  0001 C CNN
 	1    9150 1500
@@
 F 0 "L4" V 7750 4100 50  0000 C CNN
 F 1 "22uH" V 7875 4100 50  0000 C CNN
-F 2 "" H 7800 4100 50  0001 C CNN
+F 2 "Resistors_SMD:R_0805" H 7800 4100 50  0001 C CNN
 F 3 "" H 7800 4100 50  0001 C CNN
 	1    7800 4100
@@
 F 0 "D8" H 8900 4500 50  0000 C CNN
 F 1 "SS24" H 8900 4300 50  0000 C CNN
-F 2 "" H 8900 4400 50  0001 C CNN
+F 2 "SMD_Packages-Custom:DO-214AA" H 8900 4400 50  0001 C CNN
 F 3 "" H 8900 4400 50  0001 C CNN
 	1    8900 4400
@@
 F 0 "L2" V 7200 5700 50  0000 C CNN
 F 1 "22uH" V 7325 5700 50  0000 C CNN
-F 2 "" H 7250 5700 50  0001 C CNN
+F 2 "Resistors_SMD:R_0805" H 7250 5700 50  0001 C CNN
 F 3 "" H 7250 5700 50  0001 C CNN
 	1    7250 5700
@@
 F 0 "D10" H 9150 4200 50  0000 C CNN
 F 1 "SS24" H 9150 4000 50  0000 C CNN
-F 2 "" H 9150 4100 50  0001 C CNN
+F 2 "SMD_Packages-Custom:DO-214AA" H 9150 4100 50  0001 C CNN
 F 3 "" H 9150 4100 50  0001 C CNN
 	1    9150 4100
@@
 F 0 "D6" H 8350 5800 50  0000 C CNN
 F 1 "SS24" H 8350 5600 50  0000 C CNN
-F 2 "" H 8350 5700 50  0001 C CNN
+F 2 "SMD_Packages-Custom:DO-214AA" H 8350 5700 50  0001 C CNN
 F 3 "" H 8350 5700 50  0001 C CNN
 	1    8350 5700

Commit message: Created footprint for trimpot.
Parts:
- RV1: footprint (none) -> Potentiometers-Custom:TT-Electronics_Pot_23B
Changed lines of the file:
@@
 F 0 "RV1" V 1150 5100 50  0000 C CNN
 F 1 "100k" V 1250 5100 50  0000 C CNN
-F 2 "" H 1250 5100 50  0001 C CNN
+F 2 "Potentiometers-Custom:TT-Electronics_Pot_23B" H 1250 5100 50  0001 C CNN
 F 3 "" H 1250 5100 50  0001 C CNN
 	1    1250 5100

Commit message: Finished linking all component footprints.
Parts:
- BT1: footprint (none) -> Connectors-Custom:TERMINAL-BLOCK-3.5MM-2POS
- W1, W10, W11, W2, W3, W4, W5, W6, W7, W8, W9: footprint (none) -> Connectors-Custom4:TEST-POINT
Changed lines of the file:
@@
 F 0 "W10" H 9400 1650 50  0000 C CNN
 F 1 "TEST_1P" H 9400 1650 50  0001 C CNN
-F 2 "" H 9600 1450 50  0001 C CNN
+F 2 "Connectors-Custom4:TEST-POINT" H 9600 1450 50  0001 C CNN
 F 3 "" H 9600 1450 50  0001 C CNN
 	1    9400 1450
@@
 F 0 "W8" H 9200 2700 50  0000 C CNN
 F 1 "TEST_1P" H 9200 2700 50  0001 C CNN
-F 2 "" H 9400 2500 50  0001 C CNN
+F 2 "Connectors-Custom4:TEST-POINT" H 9400 2500 50  0001 C CNN
 F 3 "" H 9400 2500 50  0001 C CNN
 	1    9200 2500
@@
 F 0 "W4" H 8600 2250 50  0000 C CNN
 F 1 "TEST_1P" H 8600 2250 50  0001 C CNN
-F 2 "" H 8800 2050 50  0001 C CNN
+F 2 "Connectors-Custom4:TEST-POINT" H 8800 2050 50  0001 C CNN
 F 3 "" H 8800 2050 50  0001 C CNN
 	1    8600 2050
@@
 F 0 "W5" H 8600 2650 50  0000 C CNN
 F 1 "TEST_1P" H 8600 2650 50  0001 C CNN
-F 2 "" H 8800 2450 50  0001 C CNN
+F 2 "Connectors-Custom4:TEST-POINT" H 8800 2450 50  0001 C CNN
 F 3 "" H 8800 2450 50  0001 C CNN
 	1    8600 2450
@@
 F 0 "W2" H 6500 1650 50  0000 C CNN
 F 1 "TEST_1P" H 6500 1650 50  0001 C CNN
-F 2 "" H 6700 1450 50  0001 C CNN
+F 2 "Connectors-Custom4:TEST-POINT" H 6700 1450 50  0001 C CNN
 F 3 "" H 6700 1450 50  0001 C CNN
 	1    6500 1450
@@
 F 0 "W3" H 6500 4250 50  0000 C CNN
 F 1 "TEST_1P" H 6500 4250 50  0001 C CNN
-F 2 "" H 6700 4050 50  0001 C CNN
+F 2 "Connectors-Custom4:TEST-POINT" H 6700 4050 50  0001 C CNN
 F 3 "" H 6700 4050 50  0001 C CNN
 	1    6500 4050
@@
 F 0 "W11" H 9400 4250 50  0000 C CNN
 F 1 "TEST_1P" H 9400 4250 50  0001 C CNN
-F 2 "" H 9600 4050 50  0001 C CNN
+F 2 "Connectors-Custom4:TEST-POINT" H 9600 4050 50  0001 C CNN
 F 3 "" H 9600 4050 50  0001 C CNN
 	1    9400 4050
@@
 F 0 "W9" H 9200 5300 50  0000 C CNN
 F 1 "TEST_1P" H 9200 5300 50  0001 C CNN
-F 2 "" H 9400 5100 50  0001 C CNN
+F 2 "Connectors-Custom4:TEST-POINT" H 9400 5100 50  0001 C CNN
 F 3 "" H 9400 5100 50  0001 C CNN
 	1    9200 5100
@@
 F 0 "W6" H 8600 4850 50  0000 C CNN
 F 1 "TEST_1P" H 8600 4850 50  0001 C CNN
-F 2 "" H 8800 4650 50  0001 C CNN
+F 2 "Connectors-Custom4:TEST-POINT" H 8800 4650 50  0001 C CNN
 F 3 "" H 8800 4650 50  0001 C CNN
 	1    8600 4650
@@
 F 0 "W7" H 8600 5250 50  0000 C CNN
 F 1 "TEST_1P" H 8600 5250 50  0001 C CNN
-F 2 "" H 8800 5050 50  0001 C CNN
+F 2 "Connectors-Custom4:TEST-POINT" H 8800 5050 50  0001 C CNN
 F 3 "" H 8800 5050 50  0001 C CNN
 	1    8600 5050
@@
 F 0 "W1" H 2550 5250 50  0000 C CNN
 F 1 "TEST_1P" H 2550 5250 50  0001 C CNN
-F 2 "" H 2750 5050 50  0001 C CNN
+F 2 "Connectors-Custom4:TEST-POINT" H 2750 5050 50  0001 C CNN
 F 3 "" H 2750 5050 50  0001 C CNN
 	1    2550 5050
@@
 F 0 "BT1" H 4800 2900 50  0000 L CNN
 F 1 "3.7V Li-Ion" H 4700 2750 50  0000 L CNN
-F 2 "" V 4700 2860 50  0001 C CNN
+F 2 "Connectors-Custom:TERMINAL-BLOCK-3.5MM-2POS" V 4700 2860 50  0001 C CNN
 F 3 "" V 4700 2860 50  0001 C CNN
 	1    4700 2800
