File: EE-Ink.kicad_pcb (KiCad board)
At the start: 2 copper layers, 93 parts, among them J1 USB_A, Q1 S8050, Q2 S8050, Q3 MMUN2211, Q4 IRLML6402, Q5 IRLML6402, Q6 IRLML6402, U1 ED060SC4, U2 74LV4094, U3 ESP32-WROOM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

Commit message: Fixed footprint for S8050 transistors.
Parts:
- Q1, Q2: footprint TO_SOT_Packages_THT:TO-92_Molded_Narrow -> TO_SOT_Packages_SMD:SOT-23
Changed lines of the file:
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@@
   (general
     (links 212)
-    (no_connects 144)
+    (no_connects 212)
     (area 0 0 0 0)
     (thickness 1.6)
@@
     (pad_to_mask_clearance 0.2)
     (aux_axis_origin 0 0)
-    (visible_elements FFFFFF7F)
+    (visible_elements 7FFFFFFF)
     (pcbplotparams
       (layerselection 0x00030_80000001)
@@
     )
   )
-  (module TO_SOT_Packages_THT:TO-92_Molded_Narrow (layer F.Cu)
-    (at 183.26 123.5)
-    (descr "TO-92 leads molded, narrow, drill 0.6mm (see NXP sot054_po.pdf)")
-    (tags "to-92 sc-43 sc-43a sot54 PA33 transistor")
-    (fp_text reference Q1 (at 1.27 -3.56) (layer F.SilkS)
-      (effects (font (size 1 1) (thickness 0.15)))
-    )
-    (fp_text value S8050 (at 1.27 2.79) (layer F.Fab)
-      (effects (font (size 1 1) (thickness 0.15)))
-    )
-    (fp_text user %R (at 1.27 -3.56) (layer F.Fab)
-      (effects (font (size 1 1) (thickness 0.15)))
-    )
-    (fp_line (start -0.53 1.85) (end 3.07 1.85) (layer F.SilkS) (width 0.12))
-    (fp_line (start -0.5 1.75) (end 3 1.75) (layer F.Fab) (width 0.1))
-    (fp_line (start -1.46 -2.73) (end 4 -2.73) (layer F.CrtYd) (width 0.05))
-    (fp_line (start -1.46 -2.73) (end -1.46 2.01) (layer F.CrtYd) (width 0.05))
-    (fp_line (start 4 2.01) (end 4 -2.73) (layer F.CrtYd) (width 0.05))
-    (fp_line (start 4 2.01) (end -1.46 2.01) (layer F.CrtYd) (width 0.05))
-    (fp_arc (start 1.27 0) (end 1.27 -2.48) (angle 135) (layer F.Fab) (width 0.1))
-    (fp_arc (start 1.27 0) (end 1.27 -2.6) (angle -135) (layer F.SilkS) (width 0.12))
-    (fp_arc (start 1.27 0) (end 1.27 -2.48) (angle -135) (layer F.Fab) (width 0.1))
-    (fp_arc (start 1.27 0) (end 1.27 -2.6) (angle 135) (layer F.SilkS) (width 0.12))
-    (pad 2 thru_hole circle (at 1.27 -1.27 90) (size 1 1) (drill 0.6) (layers *.Cu *.Mask)
-      (net 34 "Net-(Q1-Pad2)"))
-    (pad 3 thru_hole circle (at 2.54 0 90) (size 1 1) (drill 0.6) (layers *.Cu *.Mask)
-      (net 3 /ESP_EN))
-    (pad 1 thru_hole rect (at 0 0 90) (size 1 1) (drill 0.6) (layers *.Cu *.Mask)
-      (net 35 /FTDI_RTS))
-    (model ${KISYS3DMOD}/TO_SOT_Packages_THT.3dshapes/TO-92_Molded_Narrow.wrl
-      (at (xyz 0.05 0 0))
-      (scale (xyz 1 1 1))
-      (rotate (xyz 0 0 -90))
-    )
-  )
-  (module TO_SOT_Packages_THT:TO-92_Molded_Narrow (layer F.Cu)
-    (at 175.56 123.5)
-    (descr "TO-92 leads molded, narrow, drill 0.6mm (see NXP sot054_po.pdf)")
-    (tags "to-92 sc-43 sc-43a sot54 PA33 transistor")
-    (fp_text reference Q2 (at 1.27 -3.56) (layer F.SilkS)
-      (effects (font (size 1 1) (thickness 0.15)))
-    )
-    (fp_text value S8050 (at 1.27 2.79) (layer F.Fab)
-      (effects (font (size 1 1) (thickness 0.15)))
-    )
-    (fp_text user %R (at 1.27 -3.56) (layer F.Fab)
-      (effects (font (size 1 1) (thickness 0.15)))
-    )
-    (fp_line (start -0.53 1.85) (end 3.07 1.85) (layer F.SilkS) (width 0.12))
-    (fp_line (start -0.5 1.75) (end 3 1.75) (layer F.Fab) (width 0.1))
-    (fp_line (start -1.46 -2.73) (end 4 -2.73) (layer F.CrtYd) (width 0.05))
-    (fp_line (start -1.46 -2.73) (end -1.46 2.01) (layer F.CrtYd) (width 0.05))
-    (fp_line (start 4 2.01) (end 4 -2.73) (layer F.CrtYd) (width 0.05))
-    (fp_line (start 4 2.01) (end -1.46 2.01) (layer F.CrtYd) (width 0.05))
-    (fp_arc (start 1.27 0) (end 1.27 -2.48) (angle 135) (layer F.Fab) (width 0.1))
-    (fp_arc (start 1.27 0) (end 1.27 -2.6) (angle -135) (layer F.SilkS) (width 0.12))
-    (fp_arc (start 1.27 0) (end 1.27 -2.48) (angle -135) (layer F.Fab) (width 0.1))
-    (fp_arc (start 1.27 0) (end 1.27 -2.6) (angle 135) (layer F.SilkS) (width 0.12))
-    (pad 2 thru_hole circle (at 1.27 -1.27 90) (size 1 1) (drill 0.6) (layers *.Cu *.Mask)
-      (net 36 "Net-(Q2-Pad2)"))
-    (pad 3 thru_hole circle (at 2.54 0 90) (size 1 1) (drill 0.6) (layers *.Cu *.Mask)
-      (net 37 /ESP_IO0))
-    (pad 1 thru_hole rect (at 0 0 90) (size 1 1) (drill 0.6) (layers *.Cu *.Mask)
-      (net 38 /FTDI_DTR))
-    (model ${KISYS3DMOD}/TO_SOT_Packages_THT.3dshapes/TO-92_Molded_Narrow.wrl
-      (at (xyz 0.05 0 0))
-      (scale (xyz 1 1 1))
-      (rotate (xyz 0 0 -90))
-    )
-  )
   (module TO_SOT_Packages_SMD:SOT-23 (layer F.Cu)
     (at 108.1 106.15)
@@
       (net 21 -20V))
   )
+  (module TO_SOT_Packages_SMD:SOT-23 (layer F.Cu)
+    (at 183.26 123.5)
+    (descr "SOT-23, Standard")
+    (tags SOT-23)
+    (attr smd)
+    (fp_text reference Q1 (at 0 -2.5) (layer F.SilkS)
+      (effects (font (size 1 1) (thickness 0.15)))
+    )
+    (fp_text value S8050 (at 0 2.5) (layer F.Fab)
+      (effects (font (size 1 1) (thickness 0.15)))
+    )
+    (fp_text user %R (at 0 0) (layer F.Fab)
+      (effects (font (size 0.5 0.5) (thickness 0.075)))
+    )
+    (fp_line (start -0.7 -0.95) (end -0.7 1.5) (layer F.Fab) (width 0.1))
+    (fp_line (start -0.15 -1.52) (end 0.7 -1.52) (layer F.Fab) (width 0.1))
+    (fp_line (start -0.7 -0.95) (end -0.15 -1.52) (layer F.Fab) (width 0.1))
+    (fp_line (start 0.7 -1.52) (end 0.7 1.52) (layer F.Fab) (width 0.1))
+    (fp_line (start -0.7 1.52) (end 0.7 1.52) (layer F.Fab) (width 0.1))
+    (fp_line (start 0.76 1.58) (end 0.76 0.65) (layer F.SilkS) (width 0.12))
+    (fp_line (start 0.76 -1.58) (end 0.76 -0.65) (layer F.SilkS) (width 0.12))
+    (fp_line (start -1.7 -1.75) (end 1.7 -1.75) (layer F.CrtYd) (width 0.05))
+    (fp_line (start 1.7 -1.75) (end 1.7 1.75) (layer F.CrtYd) (width 0.05))
+    (fp_line (start 1.7 1.75) (end -1.7 1.75) (layer F.CrtYd) (width 0.05))
+    (fp_line (start -1.7 1.75) (end -1.7 -1.75) (layer F.CrtYd) (width 0.05))
+    (fp_line (start 0.76 -1.58) (end -1.4 -1.58) (layer F.SilkS) (width 0.12))
+    (fp_line (start 0.76 1.58) (end -0.7 1.58) (layer F.SilkS) (width 0.12))
+    (pad 1 smd rect (at -1 -0.95) (size 0.9 0.8) (layers F.Cu F.Paste F.Mask)
+      (net 35 /FTDI_RTS))
+    (pad 2 smd rect (at -1 0.95) (size 0.9 0.8) (layers F.Cu F.Paste F.Mask)
+      (net 34 "Net-(Q1-Pad2)"))
+    (pad 3 smd rect (at 1 0) (size 0.9 0.8) (layers F.Cu F.Paste F.Mask)
+      (net 3 /ESP_EN))
+    (model ${KISYS3DMOD}/TO_SOT_Packages_SMD.3dshapes/SOT-23.wrl
+      (at (xyz 0 0 0))
+      (scale (xyz 1 1 1))
+      (rotate (xyz 0 0 0))
+    )
+  )
+  (module TO_SOT_Packages_SMD:SOT-23 (layer F.Cu)
+    (at 175.56 123.5)
+    (descr "SOT-23, Standard")
+    (tags SOT-23)
+    (attr smd)
+    (fp_text reference Q2 (at 0 -2.5) (layer F.SilkS)
+      (effects (font (size 1 1) (thickness 0.15)))
+    )
+    (fp_text value S8050 (at 0 2.5) (layer F.Fab)
+      (effects (font (size 1 1) (thickness 0.15)))
+    )
+    (fp_text user %R (at 0 0) (layer F.Fab)
+      (effects (font (size 0.5 0.5) (thickness 0.075)))
+    )
+    (fp_line (start -0.7 -0.95) (end -0.7 1.5) (layer F.Fab) (width 0.1))
+    (fp_line (start -0.15 -1.52) (end 0.7 -1.52) (layer F.Fab) (width 0.1))
+    (fp_line (start -0.7 -0.95) (end -0.15 -1.52) (layer F.Fab) (width 0.1))
+    (fp_line (start 0.7 -1.52) (end 0.7 1.52) (layer F.Fab) (width 0.1))
+    (fp_line (start -0.7 1.52) (end 0.7 1.52) (layer F.Fab) (width 0.1))
+    (fp_line (start 0.76 1.58) (end 0.76 0.65) (layer F.SilkS) (width 0.12))
+    (fp_line (start 0.76 -1.58) (end 0.76 -0.65) (layer F.SilkS) (width 0.12))
+    (fp_line (start -1.7 -1.75) (end 1.7 -1.75) (layer F.CrtYd) (width 0.05))
+    (fp_line (start 1.7 -1.75) (end 1.7 1.75) (layer F.CrtYd) (width 0.05))
+    (fp_line (start 1.7 1.75) (end -1.7 1.75) (layer F.CrtYd) (width 0.05))
+    (fp_line (start -1.7 1.75) (end -1.7 -1.75) (layer F.CrtYd) (width 0.05))
+    (fp_line (start 0.76 -1.58) (end -1.4 -1.58) (layer F.SilkS) (width 0.12))
+    (fp_line (start 0.76 1.58) (end -0.7 1.58) (layer F.SilkS) (width 0.12))
+    (pad 1 smd rect (at -1 -0.95) (size 0.9 0.8) (layers F.Cu F.Paste F.Mask)
+      (net 38 /FTDI_DTR))
+    (pad 2 smd rect (at -1 0.95) (size 0.9 0.8) (layers F.Cu F.Paste F.Mask)
+      (net 36 "Net-(Q2-Pad2)"))
+    (pad 3 smd rect (at 1 0) (size 0.9 0.8) (layers F.Cu F.Paste F.Mask)
+      (net 37 /ESP_IO0))
+    (model ${KISYS3DMOD}/TO_SOT_Packages_SMD.3dshapes/SOT-23.wrl
+      (at (xyz 0 0 0))
+      (scale (xyz 1 1 1))
+      (rotate (xyz 0 0 0))
+    )
+  )
 )
